Commit message: Enhance differential_drive URDF model: add collision geometries for base link, lidar, wheels, and caster joint

File: src/scoutbot_design/urdf/differential_drive.urdf (robot description, URDF)
Before this commit: robot scoutbot, 6 links, 5 joints
Links:
- link base_link: geometry collision box size=0.3 0.15 0.1; visual box size=0.3 0.15 0.1
- link caster_wheel: geometry collision sphere radius=0.02; visual sphere radius=0.02
- link left_wheel: geometry collision cylinder length=0.05 radius=0.05; visual cylinder length=0.05 radius=0.05
- link lidar_link: geometry collision cylinder length=0.05 radius=0.03; visual cylinder length=0.05 radius=0.03
- link right_wheel: geometry collision cylinder length=0.05 radius=0.05; visual cylinder length=0.05 radius=0.05
