Commit message: Refactor URDF model for scoutbot: adjust dimensions, add base footprint link, and improve joint definitions

File: src/scoutbot_design/urdf/urdf.xacro (robot description, xacro)
@@ -1,4 +1,10 @@
 <?xml version="1.0"?>
 <robot name="scoutbot">
+  <link name="base_footprint"/>
+  <joint name="base_footprint_to_base_link" type="fixed">
+    <parent link="base_footprint"/>
+    <child link="base_link"/>
+    <origin xyz="0 0 0.05" rpy="0 0 0"/>
+  </joint>
   <!-- Base box -->
   <link name="base_link">
@@ -6,7 +12,10 @@
       <origin xyz="0 0 0" rpy="0 0 0"/>
       <geometry>
-        <box size="0.5 0.15 0.1"/>   <!-- length x width x height -->
+        <box size="0.3 0.15 0.1"/>
+        <!-- length x width x height -->
       </geometry>
-      <material name="red"><color rgba="0.9 0.2 0.2 1.0"/></material>
+      <material name="red">
+        <color rgba="0.9 0.2 0.2 1.0"/>
+      </material>
     </visual>
   </link>
@@ -17,5 +26,7 @@
         <cylinder radius="0.03" length="0.05"/>
       </geometry>
-      <material name="orange"><color rgba="1.0 0.5 0.1 1.0"/></material>
+      <material name="orange">
+        <color rgba="1.0 0.5 0.1 1.0"/>
+      </material>
     </visual>
   </link>
@@ -28,9 +39,11 @@
   <link name="left_wheel">
     <visual>
-      <origin xyz="0 0 0" rpy="0 1.5708 0"/> <!-- rotate so cylinder is sideways -->
       <geometry>
-        <cylinder radius="0.035" length="0.02"/>
+        <cylinder radius="0.05" length="0.05"/>
+        <origin xyz="0 0 0" rpy="0 0 0"/>
       </geometry>
-      <material name="black"><color rgba="0.1 0.1 0.1 1.0"/></material>
+      <material name="black">
+        <color rgba="0.0 0.0 0.0 1.0" />
+      </material>
     </visual>
   </link>
@@ -38,15 +51,18 @@
     <parent link="base_link"/>
     <child link="left_wheel"/>
-    <origin xyz="0 -0.09 -0.02" rpy="0 0 0"/> <!-- position: back/left side -->
-    <axis xyz="0 1 0"/> <!-- spin around Y -->
+    <!-- <origin xyz="-0.12 0.1035 0" rpy="1.57 0 0"/> -->
+    <origin xyz="-0.12 0.1035 -0.035" rpy="1.57 0 0"/>
+    <axis xyz="0.0 0.0 1.0"/>
   </joint>
   <!-- Right wheel -->
   <link name="right_wheel">
     <visual>
-      <origin xyz="0 0 0" rpy="0 1.5708 0"/>
       <geometry>
-        <cylinder radius="0.035" length="0.02"/>
+        <cylinder radius="0.05" length="0.05"/>
+        <origin xyz="0 0 0" rpy="0 0 0"/>
       </geometry>
-      <material name="black"><color rgba="0.1 0.1 0.1 1.0"/></material>
+      <material name="black">
+        <color rgba="0.0 0.0 0.0 1.0" />
+      </material>
     </visual>
   </link>
@@ -54,6 +70,7 @@
     <parent link="base_link"/>
     <child link="right_wheel"/>
-    <origin xyz="0 0.09 -0.02" rpy="0 0 0"/> <!-- position: back/right side -->
-    <axis xyz="0 1 0"/>
+    <!-- <origin xyz="-0.12 -0.1035 0" rpy="1.57 0 0"/> -->
+    <origin xyz="-0.12 -0.1035 -0.035" rpy="1.57 0 0"/>
+    <axis xyz="0.0 0.0 1.0"/>
   </joint>
   <!-- Front caster wheel -->
@@ -63,5 +80,7 @@
         <sphere radius="0.02"/>
       </geometry>
-      <material name="grey"><color rgba="0.6 0.6 0.6 1.0"/></material>
+      <material name="grey">
+        <color rgba="0.6 0.6 0.6 1.0"/>
+      </material>
     </visual>
   </link>
@@ -69,5 +88,6 @@
     <parent link="base_link"/>
     <child link="caster_wheel"/>
-    <origin xyz="0.09 0 -0.03" rpy="0 0 0"/> <!-- front/center, near ground -->
+    <origin xyz="0.1 0 -0.067" rpy="0 0 0"/>
+    <!-- front/center, near ground -->
   </joint>
 </robot>

Commit message: Enhance URDF model: add collision geometries for base link, lidar, wheels, and caster joint

File: src/scoutbot_design/urdf/urdf.xacro (robot description, xacro)
@@ -19,4 +19,11 @@
       </material>
     </visual>
+    <collision>
+      <origin xyz="0 0 0" rpy="0 0 0"/>
+      <geometry>
+        <box size="0.3 0.15 0.1"/>
+        <!-- length x width x height -->
+      </geometry>
+    </collision>
   </link>
   <!-- Lidar -->
@@ -30,4 +37,9 @@
       </material>
     </visual>
+    <collision>
+      <geometry>
+        <cylinder radius="0.03" length="0.05"/>
+      </geometry>
+    </collision>
   </link>
   <joint name="lidar_joint" type="fixed">
@@ -47,4 +59,10 @@
       </material>
     </visual>
+    <collision>
+      <geometry>
+        <cylinder radius="0.05" length="0.05"/>
+        <origin xyz="0 0 0" rpy="0 0 0"/>
+      </geometry>
+    </collision>
   </link>
   <joint name="left_wheel_joint" type="continuous">
@@ -66,4 +84,10 @@
       </material>
     </visual>
+    <collision>
+      <geometry>
+        <cylinder radius="0.05" length="0.05"/>
+        <origin xyz="0 0 0" rpy="0 0 0"/>
+      </geometry>
+    </collision>
   </link>
   <joint name="right_wheel_joint" type="continuous">
@@ -84,4 +108,9 @@
       </material>
     </visual>
+    <collision>
+      <geometry>
+        <sphere radius="0.02"/>
+      </geometry>
+    </collision>
   </link>
   <joint name="caster_joint" type="fixed">

Commit message: Enhance URDF model: add inertial properties for base link, lidar, wheels, and caster wheel

File: src/scoutbot_design/urdf/urdf.xacro (robot description, xacro)
@@ -13,5 +13,4 @@
       <geometry>
         <box size="0.3 0.15 0.1"/>
-        <!-- length x width x height -->
       </geometry>
       <material name="red">
@@ -23,7 +22,12 @@
       <geometry>
         <box size="0.3 0.15 0.1"/>
-        <!-- length x width x height -->
       </geometry>
     </collision>
+    <inertial>
+      <origin xyz="0 0 0" rpy="0 0 0"/>
+      <mass value="1.5"/>
+      <inertia ixx="0.00344" iyy="0.01219" izz="0.01519"
+               ixy="0.0" ixz="0.0" iyz="0.0"/>
+    </inertial>
   </link>
   <!-- Lidar -->
@@ -42,4 +46,10 @@
       </geometry>
     </collision>
+    <inertial>
+      <origin xyz="0 0 0" rpy="0 0 0"/>
+      <mass value="0.05"/>
+      <inertia ixx="0.000064" iyy="0.000064" izz="0.000045"
+               ixy="0.0" ixz="0.0" iyz="0.0"/>
+    </inertial>
   </link>
   <joint name="lidar_joint" type="fixed">
@@ -65,9 +75,14 @@
       </geometry>
     </collision>
+    <inertial>
+      <origin xyz="0 0 0" rpy="0 0 0"/>
+      <mass value="0.15"/>
+      <inertia ixx="0.00019" iyy="0.00013" izz="0.00019"
+               ixy="0.0" ixz="0.0" iyz="0.0"/>
+    </inertial>
   </link>
   <joint name="left_wheel_joint" type="continuous">
     <parent link="base_link"/>
     <child link="left_wheel"/>
-    <!-- <origin xyz="-0.12 0.1035 0" rpy="1.57 0 0"/> -->
     <origin xyz="-0.12 0.1035 -0.035" rpy="1.57 0 0"/>
     <axis xyz="0.0 0.0 1.0"/>
@@ -90,9 +105,14 @@
       </geometry>
     </collision>
+    <inertial>
+      <origin xyz="0 0 0" rpy="0 0 0"/>
+      <mass value="0.15"/>
+      <inertia ixx="0.00019" iyy="0.00013" izz="0.00019"
+               ixy="0.0" ixz="0.0" iyz="0.0"/>
+    </inertial>
   </link>
   <joint name="right_wheel_joint" type="continuous">
     <parent link="base_link"/>
     <child link="right_wheel"/>
-    <!-- <origin xyz="-0.12 -0.1035 0" rpy="1.57 0 0"/> -->
     <origin xyz="-0.12 -0.1035 -0.035" rpy="1.57 0 0"/>
     <axis xyz="0.0 0.0 1.0"/>
@@ -113,10 +133,12 @@
       </geometry>
     </collision>
+    <inertial>
+      <origin xyz="0 0 0" rpy="0 0 0"/>
+      <mass value="0.05"/>
+      <inertia ixx="0.000016" iyy="0.000016" izz="0.000016"
+               ixy="0.0" ixz="0.0" iyz="0.0"/>
+    </inertial>
   </link>
   <joint name="caster_joint" type="fixed">
     <parent link="base_link"/>
-    <child link="caster_wheel"/>
-    <origin xyz="0.1 0 -0.067" rpy="0 0 0"/>
-    <!-- front/center, near ground -->
-  </joint>
-</robot>
+    <child link="caster_wheel_

Commit message: Enhance CMakeLists.txt: add launch directory to install targets; add gazebo launch file for simulation

File: src/scoutbot_design/urdf/urdf.xacro (robot description, xacro)
@@ -27,6 +27,5 @@
       <origin xyz="0 0 0" rpy="0 0 0"/>
       <mass value="1.5"/>
-      <inertia ixx="0.00344" iyy="0.01219" izz="0.01519"
-               ixy="0.0" ixz="0.0" iyz="0.0"/>
+      <inertia ixx="0.00344" iyy="0.01219" izz="0.01519" ixy="0.0" ixz="0.0" iyz="0.0"/>
     </inertial>
   </link>
@@ -49,6 +48,5 @@
       <origin xyz="0 0 0" rpy="0 0 0"/>
       <mass value="0.05"/>
-      <inertia ixx="0.000064" iyy="0.000064" izz="0.000045"
-               ixy="0.0" ixz="0.0" iyz="0.0"/>
+      <inertia ixx="0.000064" iyy="0.000064" izz="0.000045" ixy="0.0" ixz="0.0" iyz="0.0"/>
     </inertial>
   </link>
@@ -78,6 +76,5 @@
       <origin xyz="0 0 0" rpy="0 0 0"/>
       <mass value="0.15"/>
-      <inertia ixx="0.00019" iyy="0.00013" izz="0.00019"
-               ixy="0.0" ixz="0.0" iyz="0.0"/>
+      <inertia ixx="0.00019" iyy="0.00013" izz="0.00019" ixy="0.0" ixz="0.0" iyz="0.0"/>
     </inertial>
   </link>
@@ -108,6 +105,5 @@
       <origin xyz="0 0 0" rpy="0 0 0"/>
       <mass value="0.15"/>
-      <inertia ixx="0.00019" iyy="0.00013" izz="0.00019"
-               ixy="0.0" ixz="0.0" iyz="0.0"/>
+      <inertia ixx="0.00019" iyy="0.00013" izz="0.00019" ixy="0.0" ixz="0.0" iyz="0.0"/>
     </inertial>
   </link>
@@ -136,9 +132,12 @@
       <origin xyz="0 0 0" rpy="0 0 0"/>
       <mass value="0.05"/>
-      <inertia ixx="0.000016" iyy="0.000016" izz="0.000016"
-               ixy="0.0" ixz="0.0" iyz="0.0"/>
+      <inertia ixx="0.000016" iyy="0.000016" izz="0.000016" ixy="0.0" ixz="0.0" iyz="0.0"/>
     </inertial>
   </link>
   <joint name="caster_joint" type="fixed">
     <parent link="base_link"/>
-    <child link="caster_wheel_
+    <child link="caster_wheel"/>
+    <origin rpy="0 0 0" xyz="0.1 0 -0.067"/>
+    <!-- front/center, near ground -->
+  </joint>
+</robot>
